Commit message: feat(robot_description): compose dual arm hand robot

File: src/marvin_description/urdf/Marvin M6-S-L-CCS-696-V4.0 urdf.urdf (robot description, URDF)
Before this commit: robot Marvin M6-S-L-CCS-696-V4.0 urdf, 8 links, 7 joints
Links:
- link Base_L: geometry collision mesh filename=package://marvin_description/meshes/left/Base_L.STL; visual mesh filename=package://marvin_description/meshes/left/Base_L.STL
- link Link1_L: geometry collision mesh filename=package://marvin_description/meshes/left/Link1_L.STL; visual mesh filename=package://marvin_description/meshes/left/Link1_L.STL
- link Link2_L: geometry collision mesh filename=package://marvin_description/meshes/left/Link2_L.STL; visual mesh filename=package://marvin_description/meshes/left/Link2_L.STL
- link Link3_L: geometry collision mesh filename=package://marvin_description/meshes/left/Link3_L.STL; visual mesh filename=package://marvin_description/meshes/left/Link3_L.STL
- link Link4_L: geometry collision mesh filename=package://marvin_description/meshes/left/Link4_L.STL; visual mesh filename=package://marvin_description/meshes/left/Link4_L.STL
- link Link5_L: geometry collision mesh filename=package://marvin_description/meshes/left/Link5_L.STL; visual mesh filename=package://marvin_description/meshes/left/Link5_L.STL
- link Link6_L: geometry collision mesh filename=package://marvin_description/meshes/left/Link6_L.STL; visual mesh filename=package://marvin_description/meshes/left/Link6_L.STL
- link Link7_L: geometry collision mesh filename=package://marvin_description/meshes/left/Link7_L.STL; visual mesh filename=package://marvin_description/meshes/left/Link7_L.STL

File: src/marvin_description/urdf/Marvin M6-S-R-CCS-696-V4.0 urdf.urdf (robot description, URDF)
Before this commit: robot Marvin M6-S-R-CCS-696-V4.0 urdf, 8 links, 7 joints
Links:
- link Base_R: geometry collision mesh filename=package://marvin_description/meshes/right/Base_R.STL; visual mesh filename=package://marvin_description/meshes/right/Base_R.STL
- link Link1_R: geometry collision mesh filename=package://marvin_description/meshes/right/Link1_R.STL; visual mesh filename=package://marvin_description/meshes/right/Link1_R.STL
- link Link2_R: geometry collision mesh filename=package://marvin_description/meshes/right/Link2_R.STL; visual mesh filename=package://marvin_description/meshes/right/Link2_R.STL
- link Link3_R: geometry collision mesh filename=package://marvin_description/meshes/right/Link3_R.STL; visual mesh filename=package://marvin_description/meshes/right/Link3_R.STL
- link Link4_R: geometry collision mesh filename=package://marvin_description/meshes/right/Link4_R.STL; visual mesh filename=package://marvin_description/meshes/right/Link4_R.STL
- link Link5_R: geometry collision mesh filename=package://marvin_description/meshes/right/Link5_R.STL; visual mesh filename=package://marvin_description/meshes/right/Link5_R.STL
- link Link6_R: geometry collision mesh filename=package://marvin_description/meshes/right/Link6_R.STL; visual mesh filename=package://marvin_description/meshes/right/Link6_R.STL
- link Link7_R: geometry collision mesh filename=package://marvin_description/meshes/right/Link7_R.STL; visual mesh filename=package://marvin_description/meshes/right/Link7_R.STL
