Commit message: feat(robot_description): add realsense and adapter geometry

File: src/robot_description/urdf/robot.urdf (robot description, URDF)
Before this commit: robot robot, 71 links, 70 joints
Links:
- removed link main_base_link
- added link base_link, mass 76.7121781204956; collision mesh filename=package://robot_description/meshes/base_link.STL; visual mesh filename=package://robot_description/meshes/base_link.STL
- added link head_camera_accel_frame
- added link head_camera_accel_optical_frame
- added link head_camera_bottom_screw_frame
- added link head_camera_color_frame
- added link head_camera_color_optical_frame
- added link head_camera_depth_frame
- added link head_camera_depth_optical_frame
- added link head_camera_gyro_frame
- added link head_camera_gyro_optical_frame
- added link head_camera_infra1_frame
- added link head_camera_infra1_optical_frame
- added link head_camera_infra2_frame
- added link head_camera_infra2_optical_frame
- added link head_camera_link, mass 0.072; collision box size=0.02505 0.09 0.025; visual mesh filename=package://realsense2_description/meshes/d435.dae
- added link left_camera_adapter_link, mass 0.05; collision mesh filename=package://robot_description/meshes/camera_adapter_link.STL; visual mesh filename=package://robot_description/meshes/camera_adapter_link.STL
- added link left_hand_docking_link, mass 0.051956; collision mesh filename=package://robot_description/meshes/hand_docking_link.STL; visual mesh filename=package://robot_description/meshes/hand_docking_link.STL
- added link lift_platform_link, mass 2.19054926095671; collision mesh filename=package://robot_description/meshes/lift_platform_link.STL; visual mesh filename=package://robot_description/meshes/lift_platform_link.STL
- added link right_camera_adapter_link, mass 0.05; collision mesh filename=package://robot_description/meshes/camera_adapter_link.STL; visual mesh filename=package://robot_description/meshes/camera_adapter_link.STL
- added link right_hand_docking_link, mass 0.051956; collision mesh filename=package://robot_description/meshes/hand_docking_link.STL; visual mesh filename=package://robot_description/meshes/hand_docking_link.STL
Joints:
- removed joint marvin_left_to_wuji_left
- removed joint marvin_right_to_wuji_right
- added joint base_to_lift_platform: type fixed, parent base_link, child lift_platform_link, origin xyz=0.2958 0.0070867 1.0124 rpy=0 0 0
- added joint head_camera_accel_joint: type fixed, parent head_camera_link, child head_camera_accel_frame, origin xyz=-0.01174 -0.00552 0.0051 rpy=0 0 0
- added joint head_camera_accel_optical_joint: type fixed, parent head_camera_accel_frame, child head_camera_accel_optical_frame, origin xyz=0 0 0 rpy=-1.5707963267948966 0 -1.5707963267948966
- added joint head_camera_color_joint: type fixed, parent head_camera_link, child head_camera_color_frame, origin xyz=0 0.015 0 rpy=0 0 0
- added joint head_camera_color_optical_joint: type fixed, parent head_camera_color_frame, child head_camera_color_optical_frame, origin xyz=0 0 0 rpy=-1.5707963267948966 0 -1.5707963267948966
- added joint head_camera_depth_joint: type fixed, parent head_camera_link, child head_camera_depth_frame, origin xyz=0 0 0 rpy=0 0 0
- added joint head_camera_depth_optical_joint: type fixed, parent head_camera_depth_frame, child head_camera_depth_optical_frame, origin xyz=0 0 0 rpy=-1.5707963267948966 0 -1.5707963267948966
- added joint head_camera_gyro_joint: type fixed, parent head_camera_link, child head_camera_gyro_frame, origin xyz=-0.01174 -0.00552 0.0051 rpy=0 0 0
- added joint head_camera_gyro_optical_joint: type fixed, parent head_camera_gyro_frame, child head_camera_gyro_optical_frame, origin xyz=0 0 0 rpy=-1.5707963267948966 0 -1.5707963267948966
- added joint head_camera_infra1_joint: type fixed, parent head_camera_link, child head_camera_infra1_frame, origin xyz=0 0.0 0 rpy=0 0 0
- added joint head_camera_infra1_optical_joint: type fixed, parent head_camera_infra1_frame, child head_camera_infra1_optical_frame, origin xyz=0 0 0 rpy=-1.5707963267948966 0 -1.5707963267948966
- added joint head_camera_infra2_joint: type fixed, parent head_camera_link, child head_camera_infra2_frame, origin xyz=0 -0.05 0 rpy=0 0 0
- added joint head_camera_infra2_optical_joint: type fixed, parent head_camera_infra2_frame, child head_camera_infra2_optical_frame, origin xyz=0 0 0 rpy=-1.5707963267948966 0 -1.5707963267948966
- added joint head_camera_joint: type fixed, parent base_link, child head_camera_bottom_screw_frame, origin xyz=0 0 1.5 rpy=0 0 0
- added joint head_camera_link_joint: type fixed, parent head_camera_bottom_screw_frame, child head_camera_link, origin xyz=0.010600000000000002 0.0175 0.0125 rpy=0 0 0
- added joint marvin_left_to_camera_adapter: type fixed, parent Link7_L, child left_camera_adapter_link, origin xyz=0 -0.14 0 rpy=1.5708 3.1416 0
- added joint marvin_left_to_wuji_left_docking: type fixed, parent Link7_L, child left_hand_docking_link, origin xyz=0 -0.14 0 rpy=1.5708 3.1416 0
- added joint marvin_right_to_camera_adapter: type fixed, parent Link7_R, child right_camera_adapter_link, origin xyz=0 -0.14 0 rpy=1.5708 0 0
- added joint marvin_right_to_wuji_right_docking: type fixed, parent Link7_R, child right_hand_docking_link, origin xyz=0 -0.14 0 rpy=1.5708 0 0
- added joint wuji_left_docking_to_wuji_left: type fixed, parent left_hand_docking_link, child left_palm_link, origin xyz=0 0 0.02 rpy=0 0 0
- added joint wuji_right_docking_to_wuji_right: type fixed, parent right_hand_docking_link, child right_palm_link, origin xyz=0 0 0.02 rpy=0 0 0
- joint main_base_to_marvin_left: origin xyz=0 0.2 0.5 rpy=-1.5708 -1.5708 0 -> xyz=0 0.2 0.0 rpy=-1.5708 -1.5708 0; parent main_base_link -> lift_platform_link
- joint main_base_to_marvin_right: origin xyz=0 -0.2 0.5 rpy=1.5708 -1.5708 0 -> xyz=0 -0.2 0.0 rpy=1.5708 -1.5708 0; parent main_base_link -> lift_platform_link

File: src/robot_description/urdf/robot.xacro (robot description, xacro)
@@ -5,35 +5,189 @@
   <xacro:include filename="wuji_left.xacro" />
   <xacro:include filename="wuji_right.xacro" />
-  <xacro:arg name="left_arm_xyz" default="0 0.2 0.5" />
+  <xacro:include filename="$(find realsense2_description)/urdf/_d435i.urdf.xacro" />
+  <xacro:arg name="left_arm_xyz" default="0.0252 0.04725 0.065" />
   <xacro:arg name="left_arm_rpy" default="-1.5708 -1.5708 0" />
-  <xacro:arg name="right_arm_xyz" default="0 -0.2 0.5" />
+  <xacro:arg name="right_arm_xyz" default="0.0252 -0.04725 0.065" />
   <xacro:arg name="right_arm_rpy" default="1.5708 -1.5708 0" />
-  <xacro:arg name="left_hand_xyz" default="0 -0.12 0" />
+  <xacro:arg name="left_hand_xyz" default="0 -0.14 0" />
   <xacro:arg name="left_hand_rpy" default="1.5708 3.1416 0" />
-  <xacro:arg name="right_hand_xyz" default="0 -0.12 0" />
+  <xacro:arg name="right_hand_xyz" default="0 -0.14 0" />
   <xacro:arg name="right_hand_rpy" default="1.5708 0 0" />
-  <link name="main_base_link" />
+  <xacro:arg name="left_camera_adapter_xyz" default="0 -0.14 0" />
+  <xacro:arg name="left_camera_adapter_rpy" default="1.5708 3.1416 0" />
+  <xacro:arg name="right_camera_adapter_xyz" default="0 -0.14 0" />
+  <xacro:arg name="right_camera_adapter_rpy" default="1.5708 0 0" />
+  <xacro:arg name="head_camera_xyz" default="0 0 1.5" />
+  <xacro:arg name="head_camera_rpy" default="0 0 0" />
+  <xacro:macro name="wuji_docking" params="prefix">
+    <link name="${prefix}_hand_docking_link">
+      <inertial>
+        <origin xyz="0.0 0.000613 0.008094" rpy="0 0 0" />
+        <mass value="0.051956" />
+        <inertia
+          ixx="1.814727e-05"
+          ixy="-2.035277e-10"
+          ixz="8.570371e-11"
+          iyy="1.736668e-05"
+          iyz="-4.906137e-07"
+          izz="1.920788e-05" />
+      </inertial>
+      <visual>
+        <origin xyz="0 0 0" rpy="0 0 0" />
+        <geometry>
+          <mesh filename="package://robot_description/meshes/hand_docking_link.STL" />
+        </geometry>
+        <material name="">
+          <color rgba="0.792156862745098 0.819607843137255 0.933333333333333 1" />
+        </material>
+      </visual>
+      <collision>
+        <origin xyz="0 0 0" rpy="0 0 0" />
+        <geometry>
+          <mesh filename="package://robot_description/meshes/hand_docking_link.STL" />
+        </geometry>
+      </collision>
+    </link>
+  </xacro:macro>
+  <xacro:macro name="camera_adapter" params="prefix">
+    <link name="${prefix}_camera_adapter_link">
+      <inertial>
+        <origin xyz="0.008437 0 0.042705" rpy="0 0 0" />
+        <mass value="0.05" />
+        <inertia
+          ixx="1.104e-04"
+          ixy="0"
+          ixz="0"
+          iyy="9.298e-05"
+          iyz="0"
+          izz="2.343e-05" />
+      </inertial>
+      <visual>
+        <origin xyz="0 0 0" rpy="0 0 0" />
+        <geometry>
+          <mesh filename="package://robot_description/meshes/camera_adapter_link.STL" />
+        </geometry>
+        <material name="">
+          <color rgba="0.55 0.55 0.55 1" />
+        </material>
+      </visual>
+      <collision>
+        <origin xyz="0 0 0" rpy="0 0 0" />
+        <geometry>
+          <mesh filename="package://robot_description/meshes/camera_adapter_link.STL" />
+        </geometry>
+      </collision>
+    </link>
+  </xacro:macro>
+  <link name="base_link">
+    <inertial>
+      <origin xyz="0.019535879789454 -0.00155643421780804 0.215131156945254" rpy="0 0 0" />
+      <mass value="76.7121781204956" />
+      <inertia
+        ixx="1.89167840103853"
+        ixy="1.68922457076388E-05"
+        ixz="0.0146214759473055"
+        iyy="2.26695150374495"
+        iyz="-0.000157897841599557"
+        izz="2.26460805565594" />
+    </inertial>
+    <visual>
+      <origin xyz="0 0 0" rpy="0 0 0" />
+      <geometry>
+        <mesh filename="package://robot_description/meshes/base_link.STL" />
+      </geometry>
+      <material name="">
+        <color rgba="1 1 1 1" />
+      </material>
+    </visual>
+    <collision>
+      <origin xyz="0 0 0" rpy="0 0 0" />
+      <geometry>
+        <mesh filename="package://robot_description/meshes/base_link.STL" />
+      </geometry>
+    </collision>
+  </link>
+  <link name="lift_platform_link">
+    <inertial>
+      <origin xyz="-0.00393440285367647 0 0.0650000000000001" rpy="0 0 0" />
+      <mass value="2.19054926095671" />
+      <inertia
+        ixx="0.00717540506836814"
+        ixy="5.23623212722548E-19"
+        ixz="4.34336481625962E-18"
+        iyy="0.0104604851986703"
+        iyz="1.22449606321944E-18"
+        izz="0.0101784648626855" />
+    </inertial>
+    <visual>
+      <origin xyz="0 0 0" rpy="0 0 0" />
+      <geometry>
+        <mesh filename="package://robot_description/meshes/lift_platform_link.STL" />
+      </geometry>
+      <material name="">
+        <color rgba="0.776470588235294 0.756862745098039 0.737254901960784 1" />
+      </material>
+    </visual>
+    <collision>
+      <origin xyz="0 0 0" rpy="0 0 0" />
+      <geometry>
+        <mesh filename="package://robot_description/meshes/lift_platform_link.STL" />
+      </geometry>
+    </collision>
+  </link>
+  <joint name="base_to_lift_platform" type="fixed">
+    <origin xyz="0.2958 0.0070867 1.0124" rpy="0 0 0" />
+    <parent link="base_link" />
+    <child link="lift_platform_link" />
+  </joint>
+  <xacro:sensor_d435i parent="base_link" name="head_camera" use_nominal_extrinsics="true">
+    <origin xyz="$(arg head_camera_xyz)" rpy="$(arg head_camera_rpy)" />
+  </xacro:sensor_d435i>
   <xacro:marvin_left />
   <xacro:marvin_right />
   <xacro:wuji_left />
   <xacro:wuji_right />
+  <xacro:wuji_docking prefix="left" />
+  <xacro:wuji_docking prefix="right" />
+  <xacro:camera_adapter prefix="left" />
+  <xacro:camera_adapter prefix="right" />
   <joint name="main_base_to_marvin_left" type="fixed">
     <origin xyz="$(arg left_arm_xyz)" rpy="$(arg left_arm_rpy)" />
-    <parent link="main_base_link" />
+    <parent link="lift_platform_link" />
     <child link="Base_L" />
   </joint>
   <joint name="main_base_to_marvin_right" type="fixed">
     <origin xyz="$(arg right_arm_xyz)" rpy="$(arg right_arm_rpy)" />
-    <parent link="main_base_link" />
+    <parent link="lift_platform_link" />
     <child link="Base_R" />
   </joint>
-  <joint name="marvin_left_to_wuji_left" type="fixed">
+  <joint name="marvin_left_to_wuji_left_docking" type="fixed">
     <origin xyz="$(arg left_hand_xyz)" rpy="$(arg left_hand_rpy)" />
     <parent link="Link7_L" />
+    <child link="left_hand_docking_link" />
+  </joint>
+  <joint name="marvin_left_to_camera_adapter" type="fixed">
+    <origin xyz="$(arg left_camera_adapter_xyz)" rpy="$(arg left_camera_adapter_rpy)" />
+    <parent link="Link7_L" />
+    <child link="left_camera_adapter_link" />
+  </joint>
+  <joint name="wuji_left_docking_to_wuji_left" type="fixed">
+    <origin xyz="0 0 0.02" rpy="0 0 0" />
+    <parent link="left_hand_docking_link" />
     <child link="left_palm_link" />
   </joint>
-  <joint name="marvin_right_to_wuji_right" type="fixed">
+  <joint name="marvin_right_to_wuji_right_docking" type="fixed">
     <origin xyz="$(arg right_hand_xyz)" rpy="$(arg right_hand_rpy)" />
     <parent link="Link7_R" />
+    <child link="right_hand_docking_link" />
+  </joint>
+  <joint name="marvin_right_to_camera_adapter" type="fixed">
+    <origin xyz="$(arg right_camera_adapter_xyz)" rpy="$(arg right_camera_adapter_rpy)" />
+    <parent link="Link7_R" />
+    <child link="right_camera_adapter_link" />
+  </joint>
+  <joint name="wuji_right_docking_to_wuji_right" type="fixed">
+    <origin xyz="0 0 0.02" rpy="0 0 0" />
+    <parent link="right_hand_docking_link" />
     <child link="right_palm_link" />
   </joint>
