Commit message: feat(robot_description): tune camera mounts and meshes

File: src/robot_description/urdf/robot.urdf (robot description, URDF)
Before this commit: robot robot, 90 links, 89 joints
Links:
- added link left_wrist_camera_accel_frame
- added link left_wrist_camera_accel_optical_frame
- added link left_wrist_camera_bottom_screw_frame
- added link left_wrist_camera_color_frame
- added link left_wrist_camera_color_optical_frame
- added link left_wrist_camera_depth_frame
- added link left_wrist_camera_depth_optical_frame
- added link left_wrist_camera_gyro_frame
- added link left_wrist_camera_gyro_optical_frame
- added link left_wrist_camera_infra1_frame
- added link left_wrist_camera_infra1_optical_frame
- added link left_wrist_camera_infra2_frame
- added link left_wrist_camera_infra2_optical_frame
- added link left_wrist_camera_link, mass 0.072; collision box size=0.02505 0.09 0.025; visual mesh filename=package://realsense2_description/meshes/d435.dae
- added link right_wrist_camera_accel_frame
- added link right_wrist_camera_accel_optical_frame
- added link right_wrist_camera_bottom_screw_frame
- added link right_wrist_camera_color_frame
- added link right_wrist_camera_color_optical_frame
- added link right_wrist_camera_depth_frame
- added link right_wrist_camera_depth_optical_frame
- added link right_wrist_camera_gyro_frame
- added link right_wrist_camera_gyro_optical_frame
- added link right_wrist_camera_infra1_frame
- added link right_wrist_camera_infra1_optical_frame
- added link right_wrist_camera_infra2_frame
- added link right_wrist_camera_infra2_optical_frame
- added link right_wrist_camera_link, mass 0.072; collision box size=0.02505 0.09 0.025; visual mesh filename=package://realsense2_description/meshes/d435.dae
Joints:
- added joint left_wrist_camera_accel_joint: type fixed, parent left_wrist_camera_link, child left_wrist_camera_accel_frame, origin xyz=-0.01174 -0.00552 0.0051 rpy=0 0 0
- added joint left_wrist_camera_accel_optical_joint: type fixed, parent left_wrist_camera_accel_frame, child left_wrist_camera_accel_optical_frame, origin xyz=0 0 0 rpy=-1.5707963267948966 0 -1.5707963267948966
- added joint left_wrist_camera_color_joint: type fixed, parent left_wrist_camera_link, child left_wrist_camera_color_frame, origin xyz=0 0.015 0 rpy=0 0 0
- added joint left_wrist_camera_color_optical_joint: type fixed, parent left_wrist_camera_color_frame, child left_wrist_camera_color_optical_frame, origin xyz=0 0 0 rpy=-1.5707963267948966 0 -1.5707963267948966
- added joint left_wrist_camera_depth_joint: type fixed, parent left_wrist_camera_link, child left_wrist_camera_depth_frame, origin xyz=0 0 0 rpy=0 0 0
- added joint left_wrist_camera_depth_optical_joint: type fixed, parent left_wrist_camera_depth_frame, child left_wrist_camera_depth_optical_frame, origin xyz=0 0 0 rpy=-1.5707963267948966 0 -1.5707963267948966
- added joint left_wrist_camera_gyro_joint: type fixed, parent left_wrist_camera_link, child left_wrist_camera_gyro_frame, origin xyz=-0.01174 -0.00552 0.0051 rpy=0 0 0
- added joint left_wrist_camera_gyro_optical_joint: type fixed, parent left_wrist_camera_gyro_frame, child left_wrist_camera_gyro_optical_frame, origin xyz=0 0 0 rpy=-1.5707963267948966 0 -1.5707963267948966
- added joint left_wrist_camera_infra1_joint: type fixed, parent left_wrist_camera_link, child left_wrist_camera_infra1_frame, origin xyz=0 0.0 0 rpy=0 0 0
- added joint left_wrist_camera_infra1_optical_joint: type fixed, parent left_wrist_camera_infra1_frame, child left_wrist_camera_infra1_optical_frame, origin xyz=0 0 0 rpy=-1.5707963267948966 0 -1.5707963267948966
- added joint left_wrist_camera_infra2_joint: type fixed, parent left_wrist_camera_link, child left_wrist_camera_infra2_frame, origin xyz=0 -0.05 0 rpy=0 0 0
- added joint left_wrist_camera_infra2_optical_joint: type fixed, parent left_wrist_camera_infra2_frame, child left_wrist_camera_infra2_optical_frame, origin xyz=0 0 0 rpy=-1.5707963267948966 0 -1.5707963267948966
- added joint left_wrist_camera_joint: type fixed, parent left_camera_adapter_link, child left_wrist_camera_bottom_screw_frame, origin xyz=0.06206 0.01137 0.06206 rpy=0 0.785398 0
- added joint left_wrist_camera_link_joint: type fixed, parent left_wrist_camera_bottom_screw_frame, child left_wrist_camera_link, origin xyz=0.010600000000000002 0.0175 0.0125 rpy=0 0 0
- added joint right_wrist_camera_accel_joint: type fixed, parent right_wrist_camera_link, child right_wrist_camera_accel_frame, origin xyz=-0.01174 -0.00552 0.0051 rpy=0 0 0
- added joint right_wrist_camera_accel_optical_joint: type fixed, parent right_wrist_camera_accel_frame, child right_wrist_camera_accel_optical_frame, origin xyz=0 0 0 rpy=-1.5707963267948966 0 -1.5707963267948966
- added joint right_wrist_camera_color_joint: type fixed, parent right_wrist_camera_link, child right_wrist_camera_color_frame, origin xyz=0 0.015 0 rpy=0 0 0
- added joint right_wrist_camera_color_optical_joint: type fixed, parent right_wrist_camera_color_frame, child right_wrist_camera_color_optical_frame, origin xyz=0 0 0 rpy=-1.5707963267948966 0 -1.5707963267948966
- added joint right_wrist_camera_depth_joint: type fixed, parent right_wrist_camera_link, child right_wrist_camera_depth_frame, origin xyz=0 0 0 rpy=0 0 0
- added joint right_wrist_camera_depth_optical_joint: type fixed, parent right_wrist_camera_depth_frame, child right_wrist_camera_depth_optical_frame, origin xyz=0 0 0 rpy=-1.5707963267948966 0 -1.5707963267948966
- added joint right_wrist_camera_gyro_joint: type fixed, parent right_wrist_camera_link, child right_wrist_camera_gyro_frame, origin xyz=-0.01174 -0.00552 0.0051 rpy=0 0 0
- added joint right_wrist_camera_gyro_optical_joint: type fixed, parent right_wrist_camera_gyro_frame, child right_wrist_camera_gyro_optical_frame, origin xyz=0 0 0 rpy=-1.5707963267948966 0 -1.5707963267948966
- added joint right_wrist_camera_infra1_joint: type fixed, parent right_wrist_camera_link, child right_wrist_camera_infra1_frame, origin xyz=0 0.0 0 rpy=0 0 0
- added joint right_wrist_camera_infra1_optical_joint: type fixed, parent right_wrist_camera_infra1_frame, child right_wrist_camera_infra1_optical_frame, origin xyz=0 0 0 rpy=-1.5707963267948966 0 -1.5707963267948966
- added joint right_wrist_camera_infra2_joint: type fixed, parent right_wrist_camera_link, child right_wrist_camera_infra2_frame, origin xyz=0 -0.05 0 rpy=0 0 0
- added joint right_wrist_camera_infra2_optical_joint: type fixed, parent right_wrist_camera_infra2_frame, child right_wrist_camera_infra2_optical_frame, origin xyz=0 0 0 rpy=-1.5707963267948966 0 -1.5707963267948966
- added joint right_wrist_camera_joint: type fixed, parent right_camera_adapter_link, child right_wrist_camera_bottom_screw_frame, origin xyz=0.06206 0.01137 0.06206 rpy=0 0.785398 0
- added joint right_wrist_camera_link_joint: type fixed, parent right_wrist_camera_bottom_screw_frame, child right_wrist_camera_link, origin xyz=0.010600000000000002 0.0175 0.0125 rpy=0 0 0
- joint base_to_lift_platform: origin xyz=0.2958 0.0070867 1.0124 rpy=0 0 0 -> xyz=0.2958 0.0070867 1.2 rpy=0 0 0
- joint head_camera_joint: origin xyz=0 0 1.5 rpy=0 0 0 -> xyz=0.35 0.0070867 1.5 rpy=0 0.959931 0
- joint main_base_to_marvin_left: origin xyz=0 0.2 0.0 rpy=-1.5708 -1.5708 0 -> xyz=0.0252 0.04725 0.065 rpy=-1.5708 -1.5708 0
- joint main_base_to_marvin_right: origin xyz=0 -0.2 0.0 rpy=1.5708 -1.5708 0 -> xyz=0.0252 -0.04725 0.065 rpy=1.5708 -1.5708 0
- joint marvin_left_to_camera_adapter: origin xyz=0 -0.14 0 rpy=1.5708 3.1416 0 -> xyz=0 -0.1 0 rpy=0.785398 0 -1.5708
- joint marvin_left_to_wuji_left_docking: origin xyz=0 -0.14 0 rpy=1.5708 3.1416 0 -> xyz=0 -0.1 0 rpy=1.5708 1.5708 0
- joint marvin_right_to_camera_adapter: origin xyz=0 -0.14 0 rpy=1.5708 0 0 -> xyz=0 -0.1 0 rpy=-0.785398 0 -1.5708
- joint marvin_right_to_wuji_right_docking: origin xyz=0 -0.14 0 rpy=1.5708 0 0 -> xyz=0 -0.1 0 rpy=1.5708 0 0
- joint wuji_left_docking_to_wuji_left: origin xyz=0 0 0.02 rpy=0 0 0 -> xyz=0 0 0.05 rpy=0 0 -0.785398
- joint wuji_right_docking_to_wuji_right: origin xyz=0 0 0.02 rpy=0 0 0 -> xyz=0 0 0.05 rpy=0 0 -0.785398

File: src/robot_description/urdf/robot.xacro (robot description, xacro)
@@ -10,14 +10,18 @@
   <xacro:arg name="right_arm_xyz" default="0.0252 -0.04725 0.065" />
   <xacro:arg name="right_arm_rpy" default="1.5708 -1.5708 0" />
-  <xacro:arg name="left_hand_xyz" default="0 -0.14 0" />
-  <xacro:arg name="left_hand_rpy" default="1.5708 3.1416 0" />
-  <xacro:arg name="right_hand_xyz" default="0 -0.14 0" />
+  <xacro:arg name="left_hand_xyz" default="0 -0.1 0" />
+  <xacro:arg name="left_hand_rpy" default="1.5708 1.5708 0" />
+  <xacro:arg name="right_hand_xyz" default="0 -0.1 0" />
   <xacro:arg name="right_hand_rpy" default="1.5708 0 0" />
-  <xacro:arg name="left_camera_adapter_xyz" default="0 -0.14 0" />
-  <xacro:arg name="left_camera_adapter_rpy" default="1.5708 3.1416 0" />
-  <xacro:arg name="right_camera_adapter_xyz" default="0 -0.14 0" />
-  <xacro:arg name="right_camera_adapter_rpy" default="1.5708 0 0" />
-  <xacro:arg name="head_camera_xyz" default="0 0 1.5" />
-  <xacro:arg name="head_camera_rpy" default="0 0 0" />
+  <xacro:arg name="left_camera_adapter_xyz" default="0 -0.1 0" />
+  <xacro:arg name="left_camera_adapter_rpy" default="0.785398 0 -1.5708" />
+  <xacro:arg name="right_camera_adapter_xyz" default="0 -0.1 0" />
+  <xacro:arg name="right_camera_adapter_rpy" default="-0.785398 0 -1.5708" />
+  <xacro:arg name="head_camera_xyz" default="0.35 0.0070867 ${1.0124+0.3}" />
+  <xacro:arg name="head_camera_rpy" default="0 0.959931 0" />
+  <xacro:arg name="left_wrist_camera_xyz" default="0.01137 0.00 0.0885" />
+  <xacro:arg name="left_wrist_camera_rpy" default="0 0.785398 0" />
+  <xacro:arg name="right_wrist_camera_xyz" default="0.01137 0.0 0.0885" />
+  <xacro:arg name="right_wrist_camera_rpy" default="0 0.785398 0" />
   <xacro:macro name="wuji_docking" params="prefix">
     <link name="${prefix}_hand_docking_link">
@@ -141,7 +145,4 @@
     <child link="lift_platform_link" />
   </joint>
-  <xacro:sensor_d435i parent="base_link" name="head_camera" use_nominal_extrinsics="true">
-    <origin xyz="$(arg head_camera_xyz)" rpy="$(arg head_camera_rpy)" />
-  </xacro:sensor_d435i>
   <xacro:marvin_left />
   <xacro:marvin_right />
@@ -173,5 +174,5 @@
   </joint>
   <joint name="wuji_left_docking_to_wuji_left" type="fixed">
-    <origin xyz="0 0 0.02" rpy="0 0 0" />
+    <origin xyz="0 0 0.05" rpy="0 0 -0.785398" />
     <parent link="left_hand_docking_link" />
     <child link="left_palm_link" />
@@ -188,7 +189,16 @@
   </joint>
   <joint name="wuji_right_docking_to_wuji_right" type="fixed">
-    <origin xyz="0 0 0.02" rpy="0 0 0" />
+    <origin xyz="0 0 0.05" rpy="0 0 -0.785398" />
     <parent link="right_hand_docking_link" />
     <child link="right_palm_link" />
   </joint>
+  <xacro:sensor_d435i parent="base_link" name="head_camera" use_nominal_extrinsics="true">
+    <origin xyz="$(arg head_camera_xyz)" rpy="$(arg head_camera_rpy)" />
+  </xacro:sensor_d435i>
+  <xacro:sensor_d435i parent="left_camera_adapter_link" name="left_wrist_camera" use_nominal_extrinsics="true">
+    <origin xyz="$(arg left_wrist_camera_xyz)" rpy="$(arg left_wrist_camera_rpy)" />
+  </xacro:sensor_d435i>
+  <xacro:sensor_d435i parent="right_camera_adapter_link" name="right_wrist_camera" use_nominal_extrinsics="true">
+    <origin xyz="$(arg right_wrist_camera_xyz)" rpy="$(arg right_wrist_camera_rpy)" />
+  </xacro:sensor_d435i>
 </robot>

Commit message: fix(robot_description): sync head camera pose

File: src/robot_description/urdf/robot.urdf (robot description, URDF)
Before this commit: robot robot, 118 links, 117 joints
Joints:
- joint head_camera_joint: origin xyz=0.35 0.0070867 1.3124 rpy=0 0.959931 0 -> xyz=0.30 0.0070867 1.4 rpy=0 1.047198 0

File: src/robot_description/urdf/robot.xacro (robot description, xacro)
@@ -18,6 +18,6 @@
   <xacro:arg name="right_camera_adapter_xyz" default="0 -0.1 0" />
   <xacro:arg name="right_camera_adapter_rpy" default="-0.785398 0 -1.5708" />
-  <xacro:arg name="head_camera_xyz" default="0.35 0.0070867 ${1.0124+0.3}" />
-  <xacro:arg name="head_camera_rpy" default="0 0.959931 0" />
+  <xacro:arg name="head_camera_xyz" default="0.30 0.0070867 1.4" />
+  <xacro:arg name="head_camera_rpy" default="0 1.047198 0" />
   <xacro:arg name="left_wrist_camera_xyz" default="0.01137 0.00 0.0885" />
   <xacro:arg name="left_wrist_camera_rpy" default="0 0.785398 0" />
