Commit message: feat(robot_description): export mjcf with multi-camera scene

File: src/robot_description/mjcf/_robot_mujoco_input.urdf (robot description, URDF)
Before this commit: robot robot, 71 links, 70 joints
Links:
- removed link main_base_link
- added link base_link, mass 76.7121781204956; collision mesh filename=robot_description/meshes/base_link.STL; visual mesh filename=robot_description/meshes/base_link.STL
- added link head_camera_accel_frame
- added link head_camera_accel_optical_frame
- added link head_camera_bottom_screw_frame
- added link head_camera_color_frame
- added link head_camera_color_optical_frame
- added link head_camera_depth_frame
- added link head_camera_depth_optical_frame
- added link head_camera_gyro_frame
- added link head_camera_gyro_optical_frame
- added link head_camera_infra1_frame
- added link head_camera_infra1_optical_frame
- added link head_camera_infra2_frame
- added link head_camera_infra2_optical_frame
- added link head_camera_link, mass 0.072; collision box size=0.02505 0.09 0.025
- added link left_camera_adapter_link, mass 0.05; collision mesh filename=robot_description/meshes/camera_adapter_link.STL; visual mesh filename=robot_description/meshes/camera_adapter_link.STL
- added link left_hand_docking_link, mass 0.051956; collision mesh filename=robot_description/meshes/hand_docking_link.STL; visual mesh filename=robot_description/meshes/hand_docking_link.STL
- added link left_wrist_camera_accel_frame
- added link left_wrist_camera_accel_optical_frame
- added link left_wrist_camera_bottom_screw_frame
- added link left_wrist_camera_color_frame
- added link left_wrist_camera_color_optical_frame
- added link left_wrist_camera_depth_frame
- added link left_wrist_camera_depth_optical_frame
- added link left_wrist_camera_gyro_frame
- added link left_wrist_camera_gyro_optical_frame
- added link left_wrist_camera_infra1_frame
- added link left_wrist_camera_infra1_optical_frame
- added link left_wrist_camera_infra2_frame
- added link left_wrist_camera_infra2_optical_frame
- added link left_wrist_camera_link, mass 0.072; collision box size=0.02505 0.09 0.025
- added link lift_platform_link, mass 2.19054926095671; collision mesh filename=robot_description/meshes/lift_platform_link.STL; visual mesh filename=robot_description/meshes/lift_platform_link.STL
- added link right_camera_adapter_link, mass 0.05; collision mesh filename=robot_description/meshes/camera_adapter_link.STL; visual mesh filename=robot_description/meshes/camera_adapter_link.STL
- added link right_hand_docking_link, mass 0.051956; collision mesh filename=robot_description/meshes/hand_docking_link.STL; visual mesh filename=robot_description/meshes/hand_docking_link.STL
- added link right_wrist_camera_accel_frame
- added link right_wrist_camera_accel_optical_frame
- added link right_wrist_camera_bottom_screw_frame
- added link right_wrist_camera_color_frame
- added link right_wrist_camera_color_optical_frame
- added link right_wrist_camera_depth_frame
- added link right_wrist_camera_depth_optical_frame
- added link right_wrist_camera_gyro_frame
- added link right_wrist_camera_gyro_optical_frame
- added link right_wrist_camera_infra1_frame
- added link right_wrist_camera_infra1_optical_frame
- added link right_wrist_camera_infra2_frame
- added link right_wrist_camera_infra2_optical_frame
- added link right_wrist_camera_link, mass 0.072; collision box size=0.02505 0.09 0.025
Joints:
- removed joint marvin_left_to_wuji_left
- removed joint marvin_right_to_wuji_right
- added joint base_to_lift_platform: type fixed, parent base_link, child lift_platform_link, origin xyz=0.2958 0.0070867 1.0124 rpy=0 0 0
- added joint head_camera_accel_joint: type fixed, parent head_camera_link, child head_camera_accel_frame, origin xyz=-0.01174 -0.00552 0.0051 rpy=0 0 0
- added joint head_camera_accel_optical_joint: type fixed, parent head_camera_accel_frame, child head_camera_accel_optical_frame, origin xyz=0 0 0 rpy=-1.5707963267948966 0 -1.5707963267948966
- added joint head_camera_color_joint: type fixed, parent head_camera_link, child head_camera_color_frame, origin xyz=0 0.015 0 rpy=0 0 0
- added joint head_camera_color_optical_joint: type fixed, parent head_camera_color_frame, child head_camera_color_optical_frame, origin xyz=0 0 0 rpy=-1.5707963267948966 0 -1.5707963267948966
- added joint head_camera_depth_joint: type fixed, parent head_camera_link, child head_camera_depth_frame, origin xyz=0 0 0 rpy=0 0 0
- added joint head_camera_depth_optical_joint: type fixed, parent head_camera_depth_frame, child head_camera_depth_optical_frame, origin xyz=0 0 0 rpy=-1.5707963267948966 0 -1.5707963267948966
- added joint head_camera_gyro_joint: type fixed, parent head_camera_link, child head_camera_gyro_frame, origin xyz=-0.01174 -0.00552 0.0051 rpy=0 0 0
- added joint head_camera_gyro_optical_joint: type fixed, parent head_camera_gyro_frame, child head_camera_gyro_optical_frame, origin xyz=0 0 0 rpy=-1.5707963267948966 0 -1.5707963267948966
- added joint head_camera_infra1_joint: type fixed, parent head_camera_link, child head_camera_infra1_frame, origin xyz=0 0.0 0 rpy=0 0 0
- added joint head_camera_infra1_optical_joint: type fixed, parent head_camera_infra1_frame, child head_camera_infra1_optical_frame, origin xyz=0 0 0 rpy=-1.5707963267948966 0 -1.5707963267948966
- added joint head_camera_infra2_joint: type fixed, parent head_camera_link, child head_camera_infra2_frame, origin xyz=0 -0.05 0 rpy=0 0 0
- added joint head_camera_infra2_optical_joint: type fixed, parent head_camera_infra2_frame, child head_camera_infra2_optical_frame, origin xyz=0 0 0 rpy=-1.5707963267948966 0 -1.5707963267948966
- added joint head_camera_joint: type fixed, parent base_link, child head_camera_bottom_screw_frame, origin xyz=0.35 0.0070867 1.3124 rpy=0 0.959931 0
- added joint head_camera_link_joint: type fixed, parent head_camera_bottom_screw_frame, child head_camera_link, origin xyz=0.010600000000000002 0.0175 0.0125 rpy=0 0 0
- added joint left_wrist_camera_accel_joint: type fixed, parent left_wrist_camera_link, child left_wrist_camera_accel_frame, origin xyz=-0.01174 -0.00552 0.0051 rpy=0 0 0
- added joint left_wrist_camera_accel_optical_joint: type fixed, parent left_wrist_camera_accel_frame, child left_wrist_camera_accel_optical_frame, origin xyz=0 0 0 rpy=-1.5707963267948966 0 -1.5707963267948966
- added joint left_wrist_camera_color_joint: type fixed, parent left_wrist_camera_link, child left_wrist_camera_color_frame, origin xyz=0 0.015 0 rpy=0 0 0
- added joint left_wrist_camera_color_optical_joint: type fixed, parent left_wrist_camera_color_frame, child left_wrist_camera_color_optical_frame, origin xyz=0 0 0 rpy=-1.5707963267948966 0 -1.5707963267948966
- added joint left_wrist_camera_depth_joint: type fixed, parent left_wrist_camera_link, child left_wrist_camera_depth_frame, origin xyz=0 0 0 rpy=0 0 0
- added joint left_wrist_camera_depth_optical_joint: type fixed, parent left_wrist_camera_depth_frame, child left_wrist_camera_depth_optical_frame, origin xyz=0 0 0 rpy=-1.5707963267948966 0 -1.5707963267948966
- added joint left_wrist_camera_gyro_joint: type fixed, parent left_wrist_camera_link, child left_wrist_camera_gyro_frame, origin xyz=-0.01174 -0.00552 0.0051 rpy=0 0 0
- added joint left_wrist_camera_gyro_optical_joint: type fixed, parent left_wrist_camera_gyro_frame, child left_wrist_camera_gyro_optical_frame, origin xyz=0 0 0 rpy=-1.5707963267948966 0 -1.5707963267948966
- added joint left_wrist_camera_infra1_joint: type fixed, parent left_wrist_camera_link, child left_wrist_camera_infra1_frame, origin xyz=0 0.0 0 rpy=0 0 0
- added joint left_wrist_camera_infra1_optical_joint: type fixed, parent left_wrist_camera_infra1_frame, child left_wrist_camera_infra1_optical_frame, origin xyz=0 0 0 rpy=-1.5707963267948966 0 -1.5707963267948966
- added joint left_wrist_camera_infra2_joint: type fixed, parent left_wrist_camera_link, child left_wrist_camera_infra2_frame, origin xyz=0 -0.05 0 rpy=0 0 0
- added joint left_wrist_camera_infra2_optical_joint: type fixed, parent left_wrist_camera_infra2_frame, child left_wrist_camera_infra2_optical_frame, origin xyz=0 0 0 rpy=-1.5707963267948966 0 -1.5707963267948966
- added joint left_wrist_camera_joint: type fixed, parent left_camera_adapter_link, child left_wrist_camera_bottom_screw_frame, origin xyz=0.01137 0.00 0.0885 rpy=0 0.785398 0
- added joint left_wrist_camera_link_joint: type fixed, parent left_wrist_camera_bottom_screw_frame, child left_wrist_camera_link, origin xyz=0.010600000000000002 0.0175 0.0125 rpy=0 0 0
- added joint marvin_left_to_camera_adapter: type fixed, parent Link7_L, child left_camera_adapter_link, origin xyz=0 -0.1 0 rpy=0.785398 0 -1.5708
- added joint marvin_left_to_wuji_left_docking: type fixed, parent Link7_L, child left_hand_docking_link, origin xyz=0 -0.1 0 rpy=1.5708 1.5708 0
- added joint marvin_right_to_camera_adapter: type fixed, parent Link7_R, child right_camera_adapter_link, origin xyz=0 -0.1 0 rpy=-0.785398 0 -1.5708
- added joint marvin_right_to_wuji_right_docking: type fixed, parent Link7_R, child right_hand_docking_link, origin xyz=0 -0.1 0 rpy=1.5708 0 0
- added joint right_wrist_camera_accel_joint: type fixed, parent right_wrist_camera_link, child right_wrist_camera_accel_frame, origin xyz=-0.01174 -0.00552 0.0051 rpy=0 0 0
- added joint right_wrist_camera_accel_optical_joint: type fixed, parent right_wrist_camera_accel_frame, child right_wrist_camera_accel_optical_frame, origin xyz=0 0 0 rpy=-1.5707963267948966 0 -1.5707963267948966
- added joint right_wrist_camera_color_joint: type fixed, parent right_wrist_camera_link, child right_wrist_camera_color_frame, origin xyz=0 0.015 0 rpy=0 0 0
- added joint right_wrist_camera_color_optical_joint: type fixed, parent right_wrist_camera_color_frame, child right_wrist_camera_color_optical_frame, origin xyz=0 0 0 rpy=-1.5707963267948966 0 -1.5707963267948966
- added joint right_wrist_camera_depth_joint: type fixed, parent right_wrist_camera_link, child right_wrist_camera_depth_frame, origin xyz=0 0 0 rpy=0 0 0
- added joint right_wrist_camera_depth_optical_joint: type fixed, parent right_wrist_camera_depth_frame, child right_wrist_camera_depth_optical_frame, origin xyz=0 0 0 rpy=-1.5707963267948966 0 -1.5707963267948966
- added joint right_wrist_camera_gyro_joint: type fixed, parent right_wrist_camera_link, child right_wrist_camera_gyro_frame, origin xyz=-0.01174 -0.00552 0.0051 rpy=0 0 0
- added joint right_wrist_camera_gyro_optical_joint: type fixed, parent right_wrist_camera_gyro_frame, child right_wrist_camera_gyro_optical_frame, origin xyz=0 0 0 rpy=-1.5707963267948966 0 -1.5707963267948966
- added joint right_wrist_camera_infra1_joint: type fixed, parent right_wrist_camera_link, child right_wrist_camera_infra1_frame, origin xyz=0 0.0 0 rpy=0 0 0
- added joint right_wrist_camera_infra1_optical_joint: type fixed, parent right_wrist_camera_infra1_frame, child right_wrist_camera_infra1_optical_frame, origin xyz=0 0 0 rpy=-1.5707963267948966 0 -1.5707963267948966
- added joint right_wrist_camera_infra2_joint: type fixed, parent right_wrist_camera_link, child right_wrist_camera_infra2_frame, origin xyz=0 -0.05 0 rpy=0 0 0
- added joint right_wrist_camera_infra2_optical_joint: type fixed, parent right_wrist_camera_infra2_frame, child right_wrist_camera_infra2_optical_frame, origin xyz=0 0 0 rpy=-1.5707963267948966 0 -1.5707963267948966
- added joint right_wrist_camera_joint: type fixed, parent right_camera_adapter_link, child right_wrist_camera_bottom_screw_frame, origin xyz=0.01137 0.0 0.0885 rpy=0 0.785398 0
- added joint right_wrist_camera_link_joint: type fixed, parent right_wrist_camera_bottom_screw_frame, child right_wrist_camera_link, origin xyz=0.010600000000000002 0.0175 0.0125 rpy=0 0 0
- added joint wuji_left_docking_to_wuji_left: type fixed, parent left_hand_docking_link, child left_palm_link, origin xyz=0 0 0.05 rpy=0 0 -0.785398
- added joint wuji_right_docking_to_wuji_right: type fixed, parent right_hand_docking_link, child right_palm_link, origin xyz=0 0 0.05 rpy=0 0 -0.785398
- joint main_base_to_marvin_left: origin xyz=0 0.2 0.5 rpy=-1.5708 -1.5708 0 -> xyz=0.0252 0.04725 0.065 rpy=-1.5708 -1.5708 0; parent main_base_link -> lift_platform_link
- joint main_base_to_marvin_right: origin xyz=0 -0.2 0.5 rpy=1.5708 -1.5708 0 -> xyz=0.0252 -0.04725 0.065 rpy=1.5708 -1.5708 0; parent main_base_link -> lift_platform_link

File: src/robot_description/urdf/robot.urdf (robot description, URDF)
Before this commit: robot robot, 118 links, 117 joints
Joints:
- joint base_to_lift_platform: origin xyz=0.2958 0.0070867 1.2 rpy=0 0 0 -> xyz=0.2958 0.0070867 1.0124 rpy=0 0 0
- joint head_camera_joint: origin xyz=0.35 0.0070867 1.5 rpy=0 0.959931 0 -> xyz=0.35 0.0070867 1.3124 rpy=0 0.959931 0
- joint left_wrist_camera_joint: origin xyz=0.06206 0.01137 0.06206 rpy=0 0.785398 0 -> xyz=0.01137 0.00 0.0885 rpy=0 0.785398 0
- joint right_wrist_camera_joint: origin xyz=0.06206 0.01137 0.06206 rpy=0 0.785398 0 -> xyz=0.01137 0.0 0.0885 rpy=0 0.785398 0

Commit message: feat(robot_description): update platform pose and scene joints

File: src/robot_description/mjcf/_robot_mujoco_input.urdf (robot description, URDF)
Before this commit: robot robot, 118 links, 117 joints
Links:
- link lift_platform_link: mass 2.19054926095671 -> 2.05736282450439
Joints:
- joint base_to_lift_platform: origin xyz=0.2958 0.0070867 1.0124 rpy=0 0 0 -> xyz=0.29899 8.6662E-05 1.0124 rpy=0 0 0
- joint head_camera_joint: origin xyz=0.35 0.0070867 1.3124 rpy=0 0.959931 0 -> xyz=0.30 0.0070867 1.4 rpy=0 1.047198 0
- joint main_base_to_marvin_left: origin xyz=0.0252 0.04725 0.065 rpy=-1.5708 -1.5708 0 -> xyz=0.02201 0.03725 0.065 rpy=-1.5708 0 0
- joint main_base_to_marvin_right: origin xyz=0.0252 -0.04725 0.065 rpy=1.5708 -1.5708 0 -> xyz=0.02201 -0.03725 0.065 rpy=1.5708 0 0

File: src/robot_description/urdf/robot.urdf (robot description, URDF)
Before this commit: robot robot, 118 links, 117 joints
Links:
- link lift_platform_link: mass 2.19054926095671 -> 2.05736282450439
Joints:
- joint base_to_lift_platform: origin xyz=0.2958 0.0070867 1.0124 rpy=0 0 0 -> xyz=0.29899 8.6662E-05 1.0124 rpy=0 0 0
- joint main_base_to_marvin_left: origin xyz=0.0252 0.04725 0.065 rpy=-1.5708 -1.5708 0 -> xyz=0.02201 0.03725 0.065 rpy=-1.5708 0 0
- joint main_base_to_marvin_right: origin xyz=0.0252 -0.04725 0.065 rpy=1.5708 -1.5708 0 -> xyz=0.02201 -0.03725 0.065 rpy=1.5708 0 0

File: src/robot_description/urdf/robot.xacro (robot description, xacro)
@@ -6,8 +6,8 @@
   <xacro:include filename="wuji_right.xacro" />
   <xacro:include filename="$(find realsense2_description)/urdf/_d435i.urdf.xacro" />
-  <xacro:arg name="left_arm_xyz" default="0.0252 0.04725 0.065" />
-  <xacro:arg name="left_arm_rpy" default="-1.5708 -1.5708 0" />
-  <xacro:arg name="right_arm_xyz" default="0.0252 -0.04725 0.065" />
-  <xacro:arg name="right_arm_rpy" default="1.5708 -1.5708 0" />
+  <xacro:arg name="left_arm_xyz" default="0.02201 0.03725 0.065" />
+  <xacro:arg name="left_arm_rpy" default="-1.5708 0 0" />
+  <xacro:arg name="right_arm_xyz" default="0.02201 -0.03725 0.065" />
+  <xacro:arg name="right_arm_rpy" default="1.5708 0 0" />
   <xacro:arg name="left_hand_xyz" default="0 -0.1 0" />
   <xacro:arg name="left_hand_rpy" default="1.5708 1.5708 0" />
@@ -114,13 +114,13 @@
   <link name="lift_platform_link">
     <inertial>
-      <origin xyz="-0.00393440285367647 0 0.0650000000000001" rpy="0 0 0" />
-      <mass value="2.19054926095671" />
+      <origin xyz="0.00304061511493919 0 0.0650000000000002" rpy="0 0 0" />
+      <mass value="2.05736282450439" />
       <inertia
-        ixx="0.00717540506836814"
-        ixy="5.23623212722548E-19"
-        ixz="4.34336481625962E-18"
-        iyy="0.0104604851986703"
-        iyz="1.22449606321944E-18"
-        izz="0.0101784648626855" />
+        ixx="0.00557455728848934"
+        ixy="-5.98328104491412E-19"
+        ixz="-8.52857618622784E-18"
+        iyy="0.00984728397591123"
+        iyz="3.66863177774555E-21"
+        izz="0.00828511749726334" />
     </inertial>
     <visual>
@@ -141,5 +141,5 @@
   </link>
   <joint name="base_to_lift_platform" type="fixed">
-    <origin xyz="0.2958 0.0070867 1.0124" rpy="0 0 0" />
+    <origin xyz="0.29899 8.6662E-05 1.0124" rpy="0 0 0" />
     <parent link="base_link" />
     <child link="lift_platform_link" />
